File: SmoothieMachinePCB.kicad_sch (KiCad schematic)
At the start: 67 parts, among them J1 Up Button, J10 Vin, J11 LCD I2C Adapter, J12 Conn_ARM_JTAG_SWD_10, J2 Down Button, J3 Next Ingredient Button, J4 Next Recipe Button, J5 Solenoid Valve, J6 Stepper Motor 2, J7 Conn_01x05, J8 Stepper Motor 1, J9 LoadCell, Q1 SS8050, Q2 SS8050, SW1 SW_Push, SW2 SW_Push, U1 ESP32-S3-WROOM-2, U2 FSA2567MPX, U3 DRV8825PWP, U4 VN10KN3-G, U6 NAU7802SGI, U7 XL1509-3.3

Commit message: Fourth wave ordered pcb files
Parts:
- removed J7: Conn_01x05, Connector_Molex:Molex_KK-254_AE-6410-05A_1x05_P2.54mm_Vertical, symbol Connector_Generic:Conn_01x05
- removed JP1: SolderJumper_3_Open, Jumper:SolderJumper-3_P2.0mm_Open_TrianglePad1.0x1.5mm, symbol Jumper:SolderJumper_3_Open
- removed L1: 47uH/3A, Inductor_SMD:L_0805_2012Metric_Pad1.05x1.20mm_HandSolder, symbol Device:L
- added J13: Conn_01x06, Connector_Molex:Molex_KK-254_AE-6410-06A_1x06_P2.54mm_Vertical, symbol Connector_Generic:Conn_01x06
- added L2: PA4342.473NLT, PA4342.473NLT:IND_PA4342_FOOTPRINT2_PUL, symbol PA4342.473NLT:PA4342.473NLT
- added R18, R19: 0 ohm, Resistor_SMD:R_0805_2012Metric_Pad1.20x1.40mm_HandSolder, symbol Device:R
- added TP1, TP10, TP11, TP12, TP13, TP14, TP15, TP16, TP17, TP18, TP19, TP2, TP20, TP21, TP22, TP23, TP24, TP25, TP26, TP27, TP28, TP29, TP3, TP30, TP31, TP32, TP33, TP34, TP35, TP36, TP37, TP38, TP4, TP7, TP8, TP9: TestPoint, TestPoint:TestPoint_Keystone_5010-5014_Multipurpose, symbol Connector:TestPoint
- C11: footprint Capacitor_SMD:C_0805_2012Metric_Pad1.18x1.45mm_HandSolder -> UUD1C101MCL1GS:U2-I_NCH
- C2: footprint Capacitor_SMD:C_0805_2012Metric_Pad1.18x1.45mm_HandSolder -> EMK325ABJ107MM-T:CAP_EMK325AB_3P2X2P5_TAY
Connections:
- net +12V: now also TP13.1
- net AOUT1: now also TP22.1
- net AOUT1C: now also TP18.1
- net AOUT2: now also TP23.1
- net AOUT2C: now also TP20.1
- net AOUT3: now also TP26.1
- net AOUT4: now also TP27.1
- net BOUT1: now also TP24.1
- net BOUT1C: now also TP19.1
- net BOUT2: now also TP25.1
- net BOUT2C: now also TP21.1
- net BOUT3: now also TP28.1
- net BOUT4: now also TP29.1
- net CHIP_PU: now also TP9.1
- net DIR: now also TP17.1
- net DTR: now also J13.3 (Pin_3), TP36.1
- net GND: now also J13.6 (Pin_6), R18.2, TP1.1, TP10.1, TP14.1, TP2.1, TP3.1, TP30.1, TP4.1
- net MTCK: now also U1.32 (MTCK/IO39)
- net MTDI: now also U1.34 (MTDI/IO41)
- net MTDO: now also U1.33 (MTDO/IO40)
- net MTMS: now also U1.35 (MTMS/IO42)
- net RTS: now also J13.2 (Pin_2), TP35.1
- net RX: now also U1.36 (RXD0/IO44), J13.5 (Pin_5), TP38.1
- net SOLENOID_VALVE: now also TP11.1
- net STEP: now also TP16.1
- net TX: now also U1.37 (TXD0/IO43), J13.4 (Pin_4), TP37.1
- net VDD33: now also J13.1 (Pin_1), R19.1, TP15.1, TP34.1, TP7.1, TP8.1
- net at D2.1 (K), U7.2 (OUT): now also L2.2
- net at C1.1, JP2.1 (A), U7.3 (FB): now also L2.1
- net LOADCELL4: now reaches C14.1, C17.1, J9.4 (Pin_4), U6.1 (REFP), U6.16 (AVDD/LDO)
- net LOADCELL4: now also TP33.1
- net LOADCELL2: now reaches J9.2 (Pin_2), R14.1
- net LOADCELL2: now also TP31.1
- net LOADCELL3: now reaches J9.3 (Pin_3), R13.1
- net LOADCELL3: now also TP32.1
- net at R4.2: now also R18.1, R19.2
- net at D1.2 (A), J5.2 (Pin_2), U4.3 (DRAIN): now also TP12.1
Other:
- moved on the sheet: C1, D2
